Commit message: fix

File: src/cr10a/urdf/urdf_files.urdf (robot description, URDF)
Before this commit: robot cr10a_robot, 8 links, 7 joints
Links:
- link Link1: geometry collision mesh filename=package://cr10a_robot/meshes/Link1.STL; visual mesh filename=package://cr10a_robot/meshes/Link1.STL
- link Link2: geometry collision mesh filename=package://cr10a_robot/meshes/Link2.STL; visual mesh filename=package://cr10a_robot/meshes/Link2.STL
- link Link3: geometry collision mesh filename=package://cr10a_robot/meshes/Link3.STL; visual mesh filename=package://cr10a_robot/meshes/Link3.STL
- link Link4: geometry collision mesh filename=package://cr10a_robot/meshes/Link4.STL; visual mesh filename=package://cr10a_robot/meshes/Link4.STL
- link Link5: geometry collision mesh filename=package://cr10a_robot/meshes/Link5.STL; visual mesh filename=package://cr10a_robot/meshes/Link5.STL
- link Link6: geometry collision mesh filename=package://cr10a_robot/meshes/Link6.STL; visual mesh filename=package://cr10a_robot/meshes/Link6.STL
- link base_link: geometry collision mesh filename=package://cr10a_robot/meshes/base_link.STL; visual mesh filename=package://cr10a_robot/meshes/base_link.STL
